File: hardware/mp16/mp16.kicad_sch (KiCad schematic)
At the start: 161 parts, among them J2 OLED SSD1306 I2C, J3 USB-C, J4 MIDI IN, J5 MIDI OUT, J6 EXPANSION, J7 LiPo 1S (pin 1 = GND, pin 2 =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, Q1 DMG2305UX, Q2 MMBT3906, SW1 SHIFT, SW10 P9, SW11 P10, SW12 P11, SW13 P12, SW14 P13, SW15 P14, SW16 P15, SW17 P16, SW18 BOOT, SW19 RESET, SW2 P1, SW20 Power, SW3 P2, SW4 P3, SW5 P4, SW6 P5, SW7 P6, SW8 P7, SW9 P8, U1 74HC165, U10 RP2040, U11 W25Q128JV, U12 USBLC6-2SC6, U13 BQ24074, U15 MAX17048, U16 TPS22917, U17 AP2112K-3.3, U18 MT3608, U19 TLP109, U2 74HC165, U20 USBLC6-2SC6, U3 74HC165, U4 74AHCT1G125, Y1 12MHz

Commit message: BOOT and RESET side by side with labels; fixed-part list; HIDE_REFS
BOOT (SW18) and RESET (SW19) stand side by side in the lower left of the
open bottom shell's window, each named on the bottom silkscreen, the SWD
pads in a row above them (order in hardware/README.md). MIDI In parts
moved to make room. tools/pcb.py: design.HIDE_REFS hides references a
label already names. The side-view charge LED joins the parts that never
move; the battery plug may move (Samuel). Not yet routed.

Co-Authored-By: Claude Opus 5.5 <noreply@anthropic.com>
Claude-Session: https://claude.ai/code/session_01P864NL83Ce2Z2DY4mgeMiF
Parts:
- C55, C56: footprint Capacitor_SMD:C_0402_1005Metric -> Capacitor_SMD:C_0603_1608Metric; MPN (none) -> CL10A106MP8NNNC
- Y1: Note (none) -> 12 MHz, CL 10 pF, approved by Abracon for the RP2040
